File: hardware/tiny_metal_detector.sch (EAGLE design)
At the start: 0 parts

Commit message: Add updated schematic, brd, gerber files and board images.
Parts:
- added A, B, GND, VCC: (no value), wirepad:3,17/1,1
- added C1: (no value), rcl:C-EUC1206K
- added C2: 100nF, rcl:C-EUC1206K
- added D1, D2: LL4148, _hhn_diodes_smd:LL4148
- added D3: SM4007, _hhn_diodes_smd:SM4007
- added IC1: TINY13-20SU, atmel:TINY13-20SU
- added J1: AVR-ISP-6PINAVR-ISP-6PIN-SMALL-SILK, avr-isp:AVR-ISP-6PINAVR-ISP-6PIN-SMALL-SILK
- added LED1: (no value), led:LEDCHIPLED_1206
- added Q1: MOSFET-NCHANNELSMD, fets:MOSFET-NCHANNELSMD
- added R1, R3: 10k, rcl:R-EU_R1206
- added R2: 330R, rcl:R-EU_R1206
- added R4: 100k, rcl:R-TRIMM3296W
- added R5: 560R, rcl:R-EU_R1206
- added R6: 200R, rcl:R-EU_R1206
- added R7: 50k, rcl:R-EU_R1206
- added S1: DTSM-3, switch-tact-custom:DTSM-3
- added SG1: F/QMBIII, buzzer:F/QMBIII
Connections:
- new net BTN: IC1.PB3/PCINT3/CLKI/ADC3, S1.2
- new net GND: C2.2, D2.A, GND.P, IC1.GND, J1.6, LED1.C, Q1.S, R3.1, R4.A, S1.1, SG1.+
- new net MOSI: IC1.PB0/PCINT0/AIN0/OC0A/MOSI, J1.4, R4.S
- new net N$1: R6.2, SG1.-
- new net N$4: B.P, C1.2, D3.A, R1.2
- new net N$5: D3.C, Q1.D
- new net N$6: Q1.G, R2.2, R3.2
- new net N$7: LED1.A, R5.2
- new net RESET: IC1.PB5/PCINT5/!RESET!/ADC0/DW, J1.5, R7.1
- new net SENS: D1.A, D2.C, IC1.PB1/PCINT1/AIN1/OC0B/INT0/MISO, J1.1, R1.1
- new net SIG: IC1.PB4/PCINT4/ADC2, R5.1, R6.1
- new net TRIGG: IC1.PB2/PCINT2/SCK/ADC1/T0, J1.3, R2.1
- new net VCC: A.P, C1.1, C2.1, D1.C, IC1.VCC, J1.2, R4.E, R7.2, VCC.P
Other:
- note added: "v.1.1"
- note added: "Łukasz Podkalicki"
